File: Ahrar Flight Controller/Ahrar Flight Controller.kicad_pcb (KiCad board)
At the start: 4 copper layers, 183 parts, among them J1 Conn_02x08_Counter_Clockwise, J10 Conn_01x06_MountingPin, J11 Conn_01x03_MountingPin, J13 1040310811, J2 Conn_01x04, J3 Conn_01x04_MountingPin, J5 Conn_01x06_MountingPin, J6 Conn_01x06_MountingPin, J7 Conn_01x03_MountingPin, J8 Conn_01x04_MountingPin, J9 USB4105-GF-A-120, Q1 BC847, SW1 SW_SPDT, SW2 SW_Push, U2 TLV1117-33, U3 MS5611-01BA, U4 TPD2EUSB30DRTR, U5 BMP581, U7 STM32H743VIT6, U8 TPS2121, Y2 32.768KHz, Y3 25MHz

Commit message: .
Parts:
- added R1: 22, Resistor_SMD:R_0603_1608Metric, F.Cu at (210.7, 89.9)
- moved C6 134.1 mm to (236.3, 74.6)
- moved C59 123.9 mm to (230.9, 88.1)
- moved C63 123.9 mm to (230.9, 90.1)
- moved C64 123.9 mm to (230.9, 92.0)
- moved C1 123.9 mm to (225.2, 88.1)
- moved C3 123.9 mm to (225.2, 90.1)
- moved C36 123.9 mm to (225.2, 92.0)
- moved C37 123.9 mm to (225.2, 94.0)
- moved C38 123.9 mm to (225.2, 96.0)
- moved C41 123.9 mm to (228.1, 88.1)
- moved C43 123.9 mm to (228.1, 90.1)
- moved C44 123.9 mm to (228.1, 92.0)
- moved C53 123.9 mm to (228.1, 94.0)
- moved C56 123.9 mm to (228.1, 96.0)
- moved Q1 120.2 mm to (236.6, 70.8)
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Other:
- board text added: "X"
- board text added: "Y"
- board text added: "Z"

Commit message: .
Parts:
- removed C13: 2.2uF, Capacitor_SMD:C_0402_1005Metric
- removed C39, C67: 100nF, Capacitor_SMD:C_0402_1005Metric
- removed TP5, TP6, TP7, TP8: TestPoint, MountingHole:MountingHole_2.5mm_Pad_Via
- added C33: 2.2uF, Capacitor_SMD:C_0603_1608Metric, F.Cu at (65.7, 244.5)
- added H1: MountingHole_Pad, MountingHole:MountingHole_2.2mm_M2_Pad_Via, F.Cu at (284.1, 270.3)
- added H2: MountingHole_Pad, MountingHole:MountingHole_2.2mm_M2_Pad_Via, F.Cu at (284.1, 276.2)
- added H3: MountingHole_Pad, MountingHole:MountingHole_2.2mm_M2_Pad_Via, F.Cu at (284.1, 282.2)
- added H4: MountingHole_Pad, MountingHole:MountingHole_2.2mm_M2_Pad_Via, F.Cu at (284.1, 288.1)
- C10, C16, C31, C36, C37, C38, C4, C41, C43, C44, C5, C57, C6, C74, C75, C9, Logo1, R107, R108, R109, R110, R111, R13, R4, R5, R9: moved to B.Cu
- moved R31 309.2 mm to (5.73, 252.5), turned to -90 degrees
- moved C74 308.6 mm to (3.06, 246.0), turned to -90 degrees
- moved R117 307.0 mm to (11.8, 232.0), turned to 90 degrees
- moved C75 306.4 mm to (3.06, 244.1), turned to 90 degrees
- moved Logo1 305.9 mm to (97.7, 286.7), turned to 180 degrees
- moved R19 304.8 mm to (6.88, 252.3), turned to 90 degrees
- moved R4 304.7 mm to (1.60, 245.6), turned to 180 degrees
- moved R58 304.5 mm to (4.74, 252.5), turned to -90 degrees
- moved R10 303.8 mm to (-13.7, 247.4), turned to 90 degrees
- moved R9 302.9 mm to (1.60, 244.5), turned to 180 degrees
- moved R20 302.7 mm to (7.87, 252.3), turned to 90 degrees
- moved C57 302.2 mm to (21.1, 225.9), turned to 180 degrees
- moved R21 300.6 mm to (8.85, 252.3), turned to 90 degrees
- moved R14 300.2 mm to (-12.9, 244.4), turned to 180 degrees
- moved C9 300.1 mm to (21.3, 222.9), turned to 180 degrees
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Connections:
- net Net-(C10-Pad2) renamed /MCU/VCAP2
- net Net-(C5-Pad2) renamed /MCU/VCAP1
- C16 pad 1: /MCU/OSC_OUT -> /MCU/OSC_IN
- C4 pad 1: /MCU/OSC_IN -> /MCU/OSC_OUT
- R19 pad 2: SERVO4 -> ESC1
- R20 pad 2: SERVO3 -> ESC2
- R21 pad 2: SERVO2 -> ESC3
- R22 pad 2: SERVO1 -> ESC4
- R29 pad 1: ESC1 -> SERVO4
- R30 pad 1: ESC2 -> SERVO3
- R31 pad 1: ESC3 -> SERVO2
- R58 pad 1: ESC4 -> SERVO1
- Y3 pad 1: /MCU/OSC_OUT -> /MCU/OSC_IN
- Y3 pad 3: /MCU/OSC_IN -> /MCU/OSC_OUT
Routing:
- net USB_D-: track 0.00 -> 3.32 mm
- net USB_D+: track 0.00 -> 3.28 mm
- net GND: track 0.00 -> 0.65 mm, vias 0 -> 1
Other:
- board text added: "E1"
- board text added: "E2"
- board text added: "E3"
- board text added: "E4"
- board text added: "S1"
- board text added: "S2"
- board text added: "S3"
- board text added: "S4"
