File: Ahrar Flight Controller/Ahrar Flight Controller.kicad_sch (KiCad schematic)
At the start: 0 parts

Commit message: Adding previous files
Other:
- sheet MCU ports: added IMU_INT, LIDAR_SCL; removed Compass_I2C_SDA

Commit message: .
Other:
- added sheet SD-card (SD-card.kicad_sch)
- added sheet USB-c (USB-c.kicad_sch)
- sheet Connectors ports: added none; removed GPS_I2C_SCL, GPS_I2C_SDA, GPS_UART_RX, GPS_UART_TX, PWM1, PWM2, PWM3, PWM4, PWM5, PWM6, PWM7, PWM8, RF_CTS, RF_RTS, RF_RX, RF_TX, SD_SPI_MISO, SD_SPI_MOSI, SD_SPI_SCLK, SD_SPI_SS, SWDCLK, SWDIO, SWDO
- sheet MCU ports: added none; removed BARO_SPI_MISO, BARO_SPI_MOSI, BARO_SPI_SCLK, BARO_SPI_SS, Compass_I2C_SCL, GPS_UART_RX, GPS_UART_TX, IMU_INT, IMU_SPI_MISO, IMU_SPI_MOSI, IMU_SPI_SCLK, IMU_SPI_SS, LIDAR_SCL, PWM1, PWM2, PWM3, PWM4, PWM5, PWM6, PWM7, PWM8, RF_CTS, RF_RTS, RF_RX, RF_TX, SD_SPI_MISO, SD_SPI_MOSI, SD_SPI_SCLK, SD_SPI_SS, SWDCLK, SWDIO, SWO
- sheet Sensors ports: added none; removed BARO_SPI_MISO, BARO_SPI_MOSI, BARO_SPI_SCLK, BARO_SPI_SS, IMU_SPI_MISO, IMU_SPI_MOSI, IMU_SPI_SCLK, IMU_SPI_SS
- note added: "Differential pair calculations"
- note added: "JLCPCB stack-up"
- note added: "Sensors Page: Connectors page: MCU Page: - Buzzer SD Cards: Power design: - Consider Single LDO 3.3V high SSR low noise Consider more filtering - Tell Halil to buy the parts, give list - Add 3D models all components"
- note added: "What's left inshAllah: - Power circuits - Buzzer - Add accurate Current conumption calculations - Adding 3D model of components"
- note removed: "- Pull-up resistors on SPI lines - Impedance and length matching for SPI lines - UART and PWM series resistors value - 3.3V Buck converter and LDO design"
- note removed: "Add the following connections: - Analog; voltage and current measurements like the Pixhawk power module -> ADC channel - additional computer that processes images -> UART (Jetson nano, Raspberry pi - reciever for control -> FrSky X8R Receiver - Pitot Tube -> I2C (Pixhawk sensor). - Buzzer -> PWM (On the board) ---------------------- consider the following with Ethernet: - Tranciever to transmit i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"
- note removed: "Check footprint for all of the components"

Commit message: .
Other:
- note added: "What's left inshAllah: - Buzzer - Adding 3D model of components"
- note removed: "What's left inshAllah: - Power circuits - Buzzer - Add accurate Current conumption calculations - Adding 3D model of components"
Changed lines of the file:
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@@
 		)
 	)
-	(text "What's left inshAllah:\n- Power circuits\n- Buzzer\n- Add accurate Current conumption calculations\n- Adding 3D model of components\n"
+	(text "What's left inshAllah:\n- Buzzer\n- Adding 3D model of components\n"
 		(exclude_from_sim no)
-		(at -207.264 35.814 0)
+		(at -138.176 32.512 0)
 		(effects
 			(font
@@
 	(text "Sensors Page:\n\nConnectors page:\n\nMCU Page:\n- Buzzer\n\nSD Cards:\n\nPower design:\n- Consider Single LDO 3.3V high SSR low noise\nConsider more filtering\n\n\n- Tell Halil to buy the parts, give list\n- Add 3D models all components"
 		(exclude_from_sim no)
-		(at -209.296 134.874 0)
+		(at -192.024 143.764 0)
 		(effects
 			(font
@@
 	)
 	(image
-		(at 148.844 -72.898)
-		(scale 5.27444)
+		(at 148.336 -74.676)
+		(scale 5.5557)
 		(data "iVBORw0KGgoAAAANSUhEUgAAAngAAAE8CAYAAABTtszdAAAABHNCSVQICAgIfAhkiAAAF6BJREFU"
 			"eJzt3WuM3fWdHvDnjM/MeGY8THwhY+PxDWxjXAM1AWKakAukoLC7FVWdzaKwyabJGjVRAiVazIYC"

Commit message: .
Parts:
- added Logo1: Logo, Footprints:Hananou logo, symbol Connector:TestPoint
- added TP5, TP6, TP7, TP8: TestPoint, MountingHole:MountingHole_2.5mm_Pad_Via, symbol Connector:TestPoint
Connections:
- new net GND: TP5.1, TP6.1, TP7.1, TP8.1
Other:
- note added: "Logo"
- note added: "Mounting Holes"
- note removed: "Sensors Page: Connectors page: MCU Page: - Buzzer SD Cards: Power design: - Consider Single LDO 3.3V high SSR low noise Consider more filtering - Tell Halil to buy the parts, give list - Add 3D models all components"

Commit message: .
Other:
- note removed: "What's left inshAllah: - Buzzer - Adding 3D model of components"
Changed lines of the file:
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@@
 		)
 	)
-	(text "What's left inshAllah:\n- Buzzer\n- Adding 3D model of components\n"
-		(exclude_from_sim no)
-		(at -138.176 32.512 0)
-		(effects
-			(font
-				(size 5.08 5.08)
-				(thickness 1.016)
-				(bold yes)
-			)
-			(justify left)
-		)
-	)
 	(text "Mounting\nHoles"
 		(exclude_from_sim no)
@@
 	)
 	(image
-		(at 34.544 34.29)
-		(scale 1.67094)
+		(at 40.894 40.894)
+		(scale 2.14896)
 		(data "iVBORw0KGgoAAAANSUhEUgAAATwAAAE7CAYAAABAAD2+AAAABHNCSVQICAgIfAhkiAAAIABJREFU"
 			"eJzsvXmYJmV57/95nqf2erfee/aNYZgVhn0bASEgoIISDe57NGrMiXtMosbkJPqLOYjGNSoadwSD"
@@
 	)
 	(sheet
-		(at 85.598 79.502)
+		(at 85.852 93.98)
 		(size 23.368 13.716)
 		(exclude_from_sim no)
@@
 		)
 		(property "Sheetname" "USB-c"
-			(at 86.106 81.534 0)
+			(at 86.36 96.012 0)
 			(show_name no)
 			(do_not_autoplace no)
@@
 		)
 		(property "Sheetfile" "USB-c.kicad_sch"
-			(at 85.344 77.724 0)
+			(at 85.598 92.202 0)
 			(show_name no)
 			(do_not_autoplace no)
@@
 	)
 	(sheet
-		(at 58.42 101.6)
+		(at 58.674 116.078)
 		(size 21.336 13.208)
 		(exclude_from_sim no)
@@
 		)
 		(property "Sheetname" "Power"
-			(at 58.928 103.378 0)
+			(at 59.182 117.856 0)
 			(show_name no)
 			(do_not_autoplace no)
@@
 		)
 		(property "Sheetfile" "Power.kicad_sch"
-			(at 58.42 99.568 0)
+			(at 58.674 114.046 0)
 			(show_name no)
 			(do_not_autoplace no)
@@
 	)
 	(sheet
-		(at 30.48 78.486)
+		(at 30.734 92.964)
 		(size 20.066 14.224)
 		(exclude_from_sim no)
@@
 		)
 		(property "Sheetname" "MCU"
-			(at 31.242 81.026 0)
+			(at 31.496 95.504 0)
 			(show_name no)
 			(do_not_autoplace no)
@@
 		)
 		(property "Sheetfile" "MCU.kicad_sch"
-			(at 30.226 76.708 0)
+			(at 30.48 91.186 0)
 			(show_name no)
 			(do_not_autoplace no)
@@
 	)
 	(sheet
-		(at 85.598 100.33)
+		(at 85.852 114.808)
 		(size 23.876 13.716)
 		(exclude_from_sim no)
@@
 		)
 		(property "Sheetname" "SD-card"
-			(at 85.852 102.616 0)
+			(at 86.106 117.094 0)
 			(show_name no)
 			(do_not_autoplace no)
@@
 		)
 		(property "Sheetfile" "SD-card.kicad_sch"
-			(at 85.344 98.298 0)
+			(at 85.598 112.776 0)
 			(show_name no)
 			(do_not_autoplace no)
@@
 	)
 	(sheet
-		(at 57.404 78.994)
+		(at 57.658 93.472)
 		(size 20.828 13.97)
 		(exclude_from_sim no)
@@
 		)
 		(property "Sheetname" "Sensors"
-			(at 57.912 81.026 0)
+			(at 58.166 95.504 0)
 			(show_name no)
 			(do_not_autoplace no)
@@
 		)
 		(property "Sheetfile" "Sensors.kicad_sch"
-			(at 56.896 76.708 0)
+			(at 57.15 91.186 0)
 			(show_name no)
 			(do_not_autoplace no)
@@
 	)
 	(sheet
-		(at 31.242 101.854)
+		(at 31.496 116.332)
 		(size 18.542 13.208)
 		(exclude_from_sim no)
@@
 		)
 		(property "Sheetname" "Connectors"
-			(at 31.496 103.632 0)
+			(at 31.75 118.11 0)
 			(show_name no)
 			(do_not_autoplace no)
@@
 		)
 		(property "Sheetfile" "Connectors.kicad_sch"
-			(at 30.988 100.076 0)
+			(at 31.242 114.554 0)
 			(show_name no)
 			(do_not_autoplace no)

Commit message: .
Parts:
- removed Logo1: Logo, Footprints:Hananou logo, symbol Connector:TestPoint
- removed TP5, TP6, TP7, TP8: TestPoint, MountingHole:MountingHole_2.5mm_Pad_Via, symbol Connector:TestPoint
- added H1, H2, H3, H4: MountingHole_Pad, MountingHole:MountingHole_2.2mm_M2_Pad_Via, symbol Mechanical:MountingHole_Pad
- added Logo1: Hananou logo, Footprints:Hananou logo, symbol Graphic:Logo_Open_Hardware_Small
Connections:
- net GND: now also H1.1, H2.1, H3.1, H4.1
