File: Ahrar Flight Controller/Connectors.kicad_sch (KiCad schematic)
At the start: 52 parts, among them J1 Micro_SD_Card, J10 Conn_01x04, J12 Conn_01x03, J13 Conn_01x06, J14 Conn_01x03, J2 Conn_01x05, J3 Conn_01x06, J7 Conn_01x04, J8 Conn_01x04

Commit message: Adding previous files
Parts:
- removed R25, R26: 2.2K, Resistor_SMD:R_0402_1005Metric, symbol Device:R
Connections:
- net GPS_UART_RX: now also R34.1; no longer R33.1
- net GPS_UART_TX: now also R33.1; no longer R34.1
- net RF_CTS: now also J13.3 (Pin_3); no longer J13.4 (Pin_4)
- net RF_RTS: now also J13.4 (Pin_4); no longer J13.3 (Pin_3)
- net RF_RX: now also J13.5 (Pin_5); no longer J13.6 (Pin_6)
- net RF_TX: now also J13.6 (Pin_6); no longer J13.5 (Pin_5)
- net GPS_I2C_SCL renamed Compass_I2C_SCL
- net GPS_I2C_SDA renamed Compass_I2C_SDA
- net LIDAR_SCL renamed Lidar_SCL
- net LIDAR_SDA renamed Lidar_SDA
- net SWDO renamed SWO
Other:
- note added: "- GPIO pins 2.54mm - Import pins from MCU page and remove SWO - Increase input capacitance - Change PWM and Dshot to 2.54mm pins - Add pull up resistors to SD-card and series resistor on clk line - Reconsider series resistors on UART lines - Pull-pull Sd-card socket same as burocket"
- note added: "Consider 2.54mm pins"
- note added: "connect rx to tx and vice versa since uart is fucked up"
- note removed: "6"
- note removed: "8 PWM: - 8 x Solder pads or pins - Optionally consider ground connections"
- note removed: "Current estimation for 3.3V handling: - MCU -> 300mA -> Buck - IMU -> 0.88 mA -> LDO - BARO -> 1.4 mA (peak)-> LDO - GPS & Compass connection -> 50mA -> LDO - SD-card -> 20-100 mA (working) 200-300mA max -> Buck ------------------------ Worst case senario - Buck = 500mA Worst case senario - LDO = 80mA Worst case senario = 680mA - 700mA ++++======================++++ Current estimation for 5V hand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"
- note removed: "GPS & Compass connections: - SDA - GND - TX - RX - VCC - SCL"
- note removed: "RF tranciever: - TX - RX - CTS (Clear to send) - RTS (Request to send) - 5V - GND"
- note removed: "SWD: - SWDIO - SWCLK - SWDO - 3.3V - GND"
- moved on the sheet: C11, C12, C34, C39, C40, C42, C7, C9, J1, J10, J12, J13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

Commit message: .
Parts:
- removed C11, C12, C7, C9: 10uF, Capacitor_SMD:C_0603_1608Metric, symbol Device:C
- removed C34, C40, C42: 1uF, Capacitor_SMD:C_0402_1005Metric, symbol Device:C
- removed J1: Micro_SD_Card, footprints.ul_473521001:CON00878_8_MOL, symbol Connector:Micro_SD_Card
- removed J12: Conn_01x03, Connector_JST:JST_GH_SM03B-GHS-TB_1x03-1MP_P1.25mm_Horizontal, symbol Connector_Generic:Conn_01x03
- removed J2: Conn_01x05, Connector_JST:JST_GH_SM05B-GHS-TB_1x05-1MP_P1.25mm_Horizontal, symbol Connector_Generic:Conn_01x05
- removed J7, J8: Conn_01x04, Connector_JST:JST_GH_SM04B-GHS-TB_1x04-1MP_P1.25mm_Horizontal, symbol Connector_Generic:Conn_01x04
- removed PIN1, PIN10, PIN11, PIN12, PIN13, PIN14, PIN15, PIN16, PIN2, PIN3, PIN4, PIN5, PIN6, PIN7, PIN8, PIN9: SolderPoint, TestPoint:TestPoint_Pad_D1.0mm, symbol Connector:TestPoint
- removed R23, R24, R4, R9: 2.2K, Resistor_SMD:R_0402_1005Metric, symbol Device:R
- added C23, C24, C27, C29: 22uF, Capacitor_SMD:C_0805_2012Metric, symbol Device:C
- added C25, C26: 100uF, Capacitor_Tantalum_SMD:CP_EIA-6032-20_AVX-F, symbol Device:C
- added C28: 2.2uF, Capacitor_SMD:C_0603_1608Metric, symbol Device:C
- added C47, C49, C50, C51, C52: 100nF, Capacitor_SMD:C_0402_1005Metric, symbol Device:C
- added J1: Conn_02x08_Counter_Clockwise, Connector_PinHeader_2.54mm:PinHeader_2x08_P2.54mm_Horizontal, symbol Connector_Generic:Conn_02x08_Counter_Clockwise
- added J15, J16: Conn_01x04, Connector_JST:JST_GH_SM04B-GHS-TB_1x04-1MP_P1.25mm_Horizontal, symbol Connector_Generic:Conn_01x04
- added J18: Conn_01x03, Connector_JST:JST_GH_SM03B-GHS-TB_1x03-1MP_P1.25mm_Horizontal, symbol Connector_Generic:Conn_01x03
- added J2: Conn_01x04, Connector_PinHeader_2.54mm:PinHeader_1x04_P2.54mm_Vertical, symbol Connector_Generic:Conn_01x04
- added R58, R61, R62, R63: 220, Resistor_SMD:R_0402_1005Metric, symbol Device:R
- added R59, R60, R64, R65, R66: 20, Resistor_SMD:R_0402_1005Metric, symbol Device:R
- added R67, R68, R69, R70, R71, R72: 4.7k, Resistor_SMD:R_0402_1005Metric, symbol Device:R
- C39: Part Number (none) -> GRM155R71C104KA88D
- J10: footprint Connector_Molex:Molex_PicoBlade_53261-0471_1x04-1MP_P1.25mm_Horizontal -> Connector_JST:JST_GH_SM04B-GHS-TB_1x04-1MP_P1.25mm_Horizontal; Distributer Link (none) -> https://www.mouser.com.tr/en/ProductDetail/JST-Commercial/S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; Part Number (none) -> SM04B-GHS-TB(LF)(SN)
- J13: footprint footprints.5024430670:CONN_502443-06xx_MOL -> Connector_Molex:Molex_CLIK-Mate_502494-0670_1x06-1MP_P2.00mm_Horizontal; Distributer Link (none) -> https://www.mouser.com.tr/en/ProductDetail/Molex/502494-067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; Part Number (none) -> 502494-0670
- J14: Distributer Link (none) -> https://www.mouser.com.tr/en/ProductDetail/JST-Commercial/S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; Part Number (none) -> SM03B-GHS-TB(LF)(SN)
- J3: Distributer Link (none) -> https://www.e-komponent.com/connector-header-sm06b-ghs-tb?s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; Part Number (none) -> SM06B-GHS-TB
- R16, R18, R32, R33, R34: value 150 -> 220; footprint Resistor_SMD:R_0603_1608Metric -> Resistor_SMD:R_0402_1005Metric; Distributer Link https://www.ozdisan.com/p/smt-smd-ve-cip-direncler-194/roya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 -> https://www.ozdisan.com/p/smt-smd-ve-cip-direncler-194/pana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; Part Number (none) -> ERJ2RKF2200X
- R19, R20, R21, R22, R28, R29, R30, R31: value 150 -> 220; footprint Resistor_SMD:R_0603_1608Metric -> Resistor_SMD:R_0402_1005Metric; Distributer Link https://www.ozdisan.com/p/smt-smd-ve-cip-direncler-194/roya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 -> https://www.ozdisan.com/p/smt-smd-ve-cip-direncler-194/pana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; Part Number HP03W5F1500T5E -> ERJ2RKF2200X
Connections:
- net +3.3VA is gone; now on net +3.3V: J3.5 (Pin_5)
- net +3.3V: now also C23.1, C49.1, J2.1 (Pin_1), R67.1, R68.1, R69.1, R70.1, R71.1, R72.1
- net +5V: now also C24.1, C25.1, C26.1, C27.1, C28.1, C29.1, C47.1, C50.1, C51.1, C52.1, J15.3 (Pin_3)
- net Compass_I2C_SCL: now also R67.2
- net Compass_I2C_SDA: now also R68.2
- net ESC1: now also R29.1; no longer R28.1
- net ESC2: now also R30.1; no longer R29.1
- net ESC3: now also R31.1; no longer R19.1
- net ESC4: now also R58.1; no longer R20.1
- net GND: now also C23.2, C24.2, C25.2, C26.2, C27.2, C28.2, C29.2, C47.2, C49.2, C50.2, C51.2, C52.2, J1.10 (Pin_10), J1.12 (Pin_12), J1.14 (Pin_14), J1.16 (Pin_16), J1.2 (Pin_2), J1.4 (Pin_4), J1.6 (Pin_6), J1.8 (Pin_8), J15.4 (Pin_4), J16.4 (Pin_4), J18.3 (Pin_3), J2.2 (Pin_2)
- net GPIO1: now also R64.1
- net GPIO2: now also R65.1
- net GPIO3: now also R66.1
- net Lidar_SCL: now also R71.2
- net Lidar_SDA: now also R72.2
- net Pitot_I2C_SCL: now also J15.2 (Pin_2), R69.2
- net Pitot_I2C_SDA: now also J15.1 (Pin_1), R70.2
- net RF_CTS: now also R63.1; no longer J13.3 (Pin_3)
- net RF_RTS: now also R62.1; no longer J13.4 (Pin_4)
- net RF_RX: now also R61.1; no longer J13.5 (Pin_5)
- net RF_SBUS_RX: now also R28.1; no longer R32.1
- net RF_TX: now also R32.1; no longer J13.6 (Pin_6)
- net SERVO1: now also R22.2; no longer R30.1
- net SERVO2: now also R21.2; no longer R31.1
- net SERVO3: now also R20.2; no longer R21.1
- net SERVO4: now also R19.2; no longer R22.1
- net SWDCLK: now also R60.1
- net SWDIO: now also R59.1
- net at R29.2: now also J1.1 (Pin_1)
- net at J14.3 (Pin_3): now also R28.2; no longer R32.2
- net at R31.2: now also J1.5 (Pin_5)
- net at R16.2: now also J18.1 (Pin_1)
- net at R18.2: now also J18.2 (Pin_2)
- net at R30.2: now also J1.3 (Pin_3)
- new net: J1.11 (Pin_11), R21.1
- new net: J1.13 (Pin_13), R20.1
- new net: J1.15 (Pin_15), R19.1
- new net: J1.7 (Pin_7), R58.2
- new net: J1.9 (Pin_9), R22.1
- new net: J16.1 (Pin_1), R64.2
- new net: J16.2 (Pin_2), R65.2
- new net: J16.3 (Pin_3), R66.2
- new net: J13.4 (Pin_4), R62.2
- new net: J13.6 (Pin_6), R32.2
- new net: J13.5 (Pin_5), R61.2
- new net: J13.3 (Pin_3), R63.2
- new net: J2.4 (Pin_4), R60.2
- new net: J2.3 (Pin_3), R59.2
Other:
- note added: "Add capacitor"
- note added: "Connections: - 8 PWM for ESCs and Servo motors - UART for GPS with a manetometer - UART for RF tranciever to communicate with GCS - UART for Auxiliary computer - SBUS (UART Reciever) for RF Reciever - I2C for pitot tube - I2C for Compass - I2C for Lidar - SWD - SDMCC for SD card"
- note added: "Current Consumption: 3mA"
- note added: "Current Consumption: 50mA-80mA"
- note added: "MAX Current Consumption: 180mA"
- note added: "MAX Current consumption: 140mA"
- note added: "Module used: BN-880"
- note added: "Module used: Benewake TFmini Plus"
- note added: "Module used: RFD868x"
- note added: "Module used: Radiolink R12DS"
- note added: "Pixhawk PX4 Differential Airspeed Sensor"
- note added: "RF Reciever"
- note removed: "- GPIO pins 2.54mm - Import pins from MCU page and remove SWO - Increase input capacitance - Change PWM and Dshot to 2.54mm pins - Add pull up resistors to SD-card and series resistor on clk line - Reconsider series resistors on UART lines - Pull-pull Sd-card socket same as burocket"
- note removed: "Connections: - 8 PWM for ESCs and Servo motors - UART for GPS with a manetometer - UART for RF tranciever to communicate with GCS - UART for Auxiliary computer - SBUS (UART Reciever) for RF Reciever - I2C for pitot tube - I2C for Compass - I2C for Lidar - SWD - SDMCC for SD card - SPI for IMU and gyro - SPI for Baro and tempterature - 3 GPIO Outputs for RGB leds"
- note removed: "Consider 2.54mm pins"
- note removed: "Current Consumption: 300mA"
- note removed: "Reciever"
- note removed: "Resistors on UART lines"
- note removed: "SD CARD"
- note removed: "connect rx to tx and vice versa since uart is fucked up"
- moved on the sheet: J10, J13, J14, J3, R16

Commit message: .
Parts:
- removed J10, J15, J16: Conn_01x04, Connector_JST:JST_GH_SM04B-GHS-TB_1x04-1MP_P1.25mm_Horizontal, symbol Connector_Generic:Conn_01x04
- removed J13: Conn_01x06, Connector_Molex:Molex_CLIK-Mate_502494-0670_1x06-1MP_P2.00mm_Horizontal, symbol Connector_Generic:Conn_01x06
- removed J14, J18: Conn_01x03, Connector_JST:JST_GH_SM03B-GHS-TB_1x03-1MP_P1.25mm_Horizontal, symbol Connector_Generic:Conn_01x03
- removed J3: Conn_01x06, Connector_JST:JST_GH_SM06B-GHS-TB_1x06-1MP_P1.25mm_Horizontal, symbol Connector_Generic:Conn_01x06
- removed R59, R60, R64, R65, R66: 20, Resistor_SMD:R_0402_1005Metric, symbol Device:R
- added J11, J7: Conn_01x03_MountingPin, Connector_JST:JST_GH_SM03B-GHS-TB_1x03-1MP_P1.25mm_Horizontal, symbol Connector_Generic_MountingPin:Conn_01x03_MountingPin
- added J3, J8: Conn_01x04_MountingPin, Connector_JST:JST_GH_SM04B-GHS-TB_1x04-1MP_P1.25mm_Horizontal, symbol Connector_Generic_MountingPin:Conn_01x04_MountingPin
- added J5: Conn_01x06_MountingPin, Connector_Molex:Molex_CLIK-Mate_502494-0670_1x06-1MP_P2.00mm_Horizontal, symbol Connector_Generic_MountingPin:Conn_01x06_MountingPin
- added J6: Conn_01x06_MountingPin, Connector_JST:JST_GH_SM06B-GHS-TB_1x06-1MP_P1.25mm_Horizontal, symbol Connector_Generic_MountingPin:Conn_01x06_MountingPin
- added R101, R102, R103, R104, R105: 22, Resistor_SMD:R_0402_1005Metric, symbol Device:R
- added TP1, TP2, TP3, TP4: TestPoint, TestPoint:TestPoint_Pad_1.0x1.0mm, symbol Connector:TestPoint
Connections:
- net +3.3V: now also J6.5 (Pin_5)
- net +5V: now also J3.1 (Pin_1), J5.1 (Pin_1), J7.3 (Pin_3), J8.3 (Pin_3)
- net Compass_I2C_SCL: now also J6.6 (Pin_6)
- net Compass_I2C_SDA: now also J6.1 (Pin_1)
- net GND: now also J11.3 (Pin_3), J11.MP (MountPin), J3.4 (Pin_4), J3.MP (MountPin), J5.2 (Pin_2), J5.MP (MountPin), J6.2 (Pin_2), J6.MP (MountPin), J7.2 (Pin_2), J7.MP (MountPin), J8.4 (Pin_4), J8.MP (MountPin), TP4.1
- net GPIO1: now also R103.1
- net GPIO2: now also R104.1
- net GPIO3: now also R105.1
- net Lidar_SCL: now also J3.3 (Pin_3)
- net Lidar_SDA: now also J3.2 (Pin_2)
- net Pitot_I2C_SCL: now also J8.2 (Pin_2)
- net Pitot_I2C_SDA: now also J8.1 (Pin_1)
- net SWDCLK: now also R102.1
- net SWDIO: now also R101.1
- net at R16.2: now also J11.1 (Pin_1)
- net at R18.2: now also J11.2 (Pin_2)
- net at R62.2: now also J5.4 (Pin_4)
- net at R28.2: now also J7.1 (Pin_1)
- net at R33.2: now also J6.4 (Pin_4)
- net at R32.2: now also J5.6 (Pin_6)
- net at R61.2: now also J5.5 (Pin_5)
- net at R34.2: now also J6.3 (Pin_3)
- net at R63.2: now also J5.3 (Pin_3)
- net at J2.4 (Pin_4): now also R102.2
- net at J2.3 (Pin_3): now also R101.2
- new net: R103.2, TP1.1
- new net: R105.2, TP3.1
- new net: R104.2, TP2.1
Other:
- note removed: "Add capacitor"
- moved on the sheet: R16, R18, R32, R61, R62, R63, R69, R70, R71, R72

Commit message: .
Parts:
- removed C39: 100nF, Capacitor_SMD:C_0402_1005Metric, symbol Device:C
Connections:
- net ESC1: now also R19.2; no longer R29.1
- net ESC2: now also R20.2; no longer R30.1
- net ESC3: now also R21.2; no longer R31.1
- net ESC4: now also R22.2; no longer R58.1
- net SERVO1: now also R58.1; no longer R22.2
- net SERVO2: now also R31.1; no longer R21.2
- net SERVO3: now also R30.1; no longer R20.2
- net SERVO4: now also R29.1; no longer R19.2
Other:
- moved on the sheet: TP2, TP3
