File: Ahrar Flight Controller/MCU.kicad_sch (KiCad schematic)
At the start: 32 parts, among them SW1 SW_SPDT, SW2 SW_Push, U7 STM32H743VIT6, Y1 25MHz

Commit message: Adding previous files
Parts:
- removed C45: 1uF, Capacitor_SMD:C_0402_1005Metric, symbol Device:C
Connections:
- net BLUE_LED: no longer D4.2 (A), D5.2 (A), U7.16 (PC1), U7.17 (PC2_C)
- net BARO_SPI_SCLK renamed BARO_SPI_CLK
- net LIDAR_SCL renamed Lidar_SCL
- net LIDAR_SDA renamed Lidar_SDA
- net SD_CK renamed SDIO_SCK
- net SD_CMD renamed SDIO_CMD
- net SD_D0 renamed SDIO_D0
- net SD_D1 renamed SDIO_D1
- net SD_D2 renamed SDIO_D2
- net SD_D3 renamed SDIO_D3
- new net GREEN_LED: D5.2 (A), U7.17 (PC2_C)
- new net RED_LED: D4.2 (A), U7.16 (PC1)
Other:
- note added: "- 4 SPI - SDMMC - 3 I2C - 1 SBUS - 3 UART - SWD - 4 Dshot - 4 PWM - 2 Channel ADC"
- note added: "- Adjust pins according to STM32CubeMX - Consider a buzzer - Add a LSE oscillator 32.768 Hz - Select ferrite bead for analog"
- note added: "Oscillator"
- note removed: "- 3 SPI - 1 I2C - 1 SWD - 2 UART - 8 PWM - 1 ADC for voltage reading - USB-c"
- moved on the sheet: D4, D5, D6, R11, R12, R14

Commit message: .
Parts:
- removed C28, C32: 1uF, Capacitor_SMD:C_0402_1005Metric, symbol Device:C
- removed D5: GREEN_LED, Capacitor_SMD:C_0603_1608Metric, symbol Device:LED
- removed R1: 47Ω, Capacitor_SMD:C_0402_1005Metric, symbol Device:R
- removed R12: 1k, Capacitor_SMD:C_0402_1005Metric, symbol Device:R
- removed R27: 10kΩ, Resistor_SMD:R_0603_1608Metric, symbol Device:R
- added C1: 6pF, Capacitor_SMD:C_0402_1005Metric, symbol Device:C
- added C16: 10pF, Capacitor_SMD:C_0603_1608Metric, symbol Device:C
- added C17, C18: 2.2uF, Capacitor_SMD:C_0603_1608Metric, symbol Device:C
- added R15: 10kΩ, Capacitor_SMD:C_0402_1005Metric, symbol Device:R
- added R24: 20, Resistor_SMD:R_0402_1005Metric, symbol Device:R
- added Y2: 32.768KHz, Crystal:Crystal_SMD_2012-2Pin_2.0x1.2mm_HandSoldering, symbol Device:Crystal
- C10, C5: footprint Capacitor_SMD:C_0402_1005Metric -> Capacitor_SMD:C_0603_1608Metric; Distributer Link https://www.ozdisan.com/p/smt-smd-ve-mlcc-kapasitorler-184/murata-grt155c81a225me13d-624222 -> https://www.ozdisan.com/p/smt-smd-ve-mlcc-kapasitorler-184/samsung-cl10b225kp8nnnc-359581?catSequenceId=184; Part Number GRT155C81A225ME13D -> CL10B225KP8NNNC
- C3: value 20pF -> 6pF; footprint Capacitor_SMD:C_0603_1608Metric -> Capacitor_SMD:C_0402_1005Metric; Distributer Link https://www.ozdisan.com/p/smt-smd-ve-mlcc-kapasitorler-184/yageo-cc0603jrnpo9bn200-747236 -> https://www.ozdisan.com/p/smt-smd-ve-mlcc-kapasitorler-184/yageo-cc0402drnpo9bn6r0-746529?catSequenceId=184; Part Number CC0603JRNPO9BN200 -> CC0402DRNPO9BN6R0
- C4: value 20pF -> 10pF; Distributer Link https://www.ozdisan.com/p/smt-smd-ve-mlcc-kapasitorler-184/yageo-cc0603jrnpo9bn200-747236 -> https://www.ozdisan.com/p/smt-smd-ve-mlcc-kapasitorler-184/samsung-cl10c100jb81pnc-522432?catSequenceId=184; Part Number CC0603JRNPO9BN200 -> CL10C100JB81PNC
- C6: value 10uF -> 22uF; Distributer Link https://www.ozdisan.com/p/tantal-kapasitorler-178/kyocera-a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 -> https://www.ozdisan.com/p/smt-smd-ve-mlcc-kapasitorler-184/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; Part Number TAJR106K006RNJ -> CL21A226KOQNNNE
- D4, D6: footprint Capacitor_SMD:C_0603_1608Metric -> LED_SMD:LED_0603_1608Metric
- FB1: footprint Resistor_SMD:R_0805_2012Metric -> Resistor_SMD:R_0603_1608Metric; Distributer Link https://www.ozdisan.com/p/bead-feritler-469/murata-blm21pg3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 -> https://www.e-komponent.com/blm18he601sn1d-murata-electroni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; Part Number (none) -> BLM18HE601SN1D
- R10: Distributer Link https://www.ozdisan.com/p/smt-smd-ve-cip-direncler-194/royalohm-0402wgj0103tce-362331 -> https://www.ozdisan.com/p/smt-smd-ve-cip-direncler-194/royalohm-cq02wgj0103tce-587874?catSequenceId=194; Part Number (none) -> CQ02WGJ0103TCE
- R11, R14: Distributer Link https://www.ozdisan.com/p/smt-smd-ve-cip-direncler-194/royalohm-hp02waf1001tce-603902 -> https://www.ozdisan.com/p/smt-smd-ve-cip-direncler-194/royalohm-0402wgj0102tce-431887?catSequenceId=194; Part Number HP02WAF1001TCE -> 0402WGJ0102TCE
- SW2: Distributer Link https://www.ozdisan.com/p/tact-sivicler-485/littelfuse-ck-k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 -> https://www.ozdisan.com/p/tact-sivicler-485/littelfuse-ck-p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; Part Number (none) -> PTS810 SJM 250 SMTR LFS
- Y1: footprint Oscillator:Oscillator_SMD_Abracon_ASE-4Pin_3.2x2.5mm -> Oscillator:Oscillator_SMD_Abracon_ASDMB-4Pin_2.5x2.0mm; Distributer Link https://www.ozdisan.com/p/osilatorler-510/raltron-com1305-2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 -> https://www.ozdisan.com/p/kristaller-508/ecs-ecs-250-10-36q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; Part Number (none) -> ECS-250-10-36Q-ES-TR
Connections:
- net GREEN_LED is gone; now on net Voltage_sense: U7.17 (PC2_C)
- net +3.3V: now also FB1.2, C17.1, C18.1, R24.2
- net +3.3VA: now also C56.1, FB1.1; no longer FB1.2
- net AUX_RX: now also U7.93 (PB7); no longer U7.64 (PC7)
- net AUX_TX: now also U7.92 (PB6); no longer U7.63 (PC6)
- net BLUE_LED: now also U7.16 (PC1); no longer U7.18 (PC3_C)
- net Boot: now also R15.1
- net Compass_I2C_SCL: now also U7.95 (PB8); no longer U7.59 (PD12)
- net Compass_I2C_SDA: now also U7.96 (PB9); no longer U7.60 (PD13)
- net Current_sense: now also U7.18 (PC3_C); no longer U7.32 (PC4)
- net GND: now also R11.2, C1.2, C16.2, C17.2, C18.2; no longer R11.1
- net GPIO1: now also U7.85 (PD4); no longer U7.7 (PC13)
- net GPIO2: now also U7.86 (PD5); no longer U7.8 (PC14)
- net GPIO3: now also U7.87 (PD6); no longer U7.9 (PC15)
- net GPS_UART_RX: now also U7.97 (PE0); no longer U7.56 (PD9)
- net GPS_UART_TX: now also U7.98 (PE1); no longer U7.55 (PD8)
- net Lidar_SCL: now also U7.59 (PD12); no longer U7.46 (PB10)
- net Lidar_SDA: now also U7.60 (PD13); no longer U7.47 (PB11)
- net OSC_OUT: now also C16.1; no longer C3.1
- net Pitot_I2C_SCL: now also U7.46 (PB10); no longer U7.92 (PB6)
- net Pitot_I2C_SDA: now also U7.47 (PB11); no longer U7.93 (PB7)
- net RED_LED: now also U7.15 (PC0); no longer U7.16 (PC1)
- net RF_SBUS_RX: now also U7.56 (PD9); no longer U7.95 (PB8)
- net SERVO3: now also U7.61 (PD14); no longer U7.53 (PB14)
- net SERVO4: now also U7.62 (PD15); no longer U7.54 (PB15)
- net VREF+: now also R24.1
- net Voltage_sense: no longer U7.33 (PC5)
- net at C59.1, SW1.2 (B): now also R15.2
- net at D4.1 (K): now also R11.1; no longer R11.2
- net BMP_INT: now reaches U7.2 (PE3)
- net ICM88_SS: now reaches U7.51 (PB12)
- net ICM88_SCK: now reaches U7.52 (PB13)
- net SD_CD: now reaches U7.82 (PD1)
- net MS_SPI_SS: now reaches U7.88 (PD7)
- net MS_SPI_MISO: now reaches U7.90 (PB4)
- net MS_SPI_MOSI: now reaches U7.91 (PB5)
- net BARO_SPI_CLK renamed BMP_SCK
- net BARO_SPI_MISO renamed BMP_MISO
- net BARO_SPI_MOSI renamed BMP_MOSI
- net BARO_SPI_SS renamed BMP_SS
- net IMU_INT: no longer names the net of U7.36 (PB2)
- net IMU_SPI_MISO renamed ICM86_MISO
- net IMU_SPI_MOSI renamed ICM86_MOSI
- net IMU_SPI_SCLK renamed ICM86_SCLK
- net IMU_SPI_SS renamed ICM86_INT
- net SWO renamed MS_SPI_CLK
- new net Buzzer: U7.63 (PC6)
- new net ICM86_SS: U7.32 (PC4)
- new net ICM88_INT: U7.55 (PD8)
- new net ICM88_MISO: U7.53 (PB14)
- new net ICM88_MOSI: U7.54 (PB15)
- new net OSC_32_IN: C1.1, U7.8 (PC14), Y2.1
- new net OSC_32_OUT: C3.1, U7.9 (PC15), Y2.2
- no-connect marks 29 -> 16
Other:
- note added: "C1 = C2 = 2(CL - Cs) ----------------- C1 = C2 = 2(10-5) = 10pF"
- note added: "C1 = C2 = 2(CL - Cs) ----------------- C1 = C2 = 2(7-4) = 6pF"
- note added: "HSE Oscillator"
- note added: "LEDs"
- note added: "LSE Oscillator"
- note added: "Max current consumption: 160mA"
- note removed: "- Adjust pins according to STM32CubeMX - Consider a buzzer - Add a LSE oscillator 32.768 Hz - Select ferrite bead for analog"
- note removed: "BUZZER RGB LEDS"
- note removed: "C1 = C2 = 2(CL - Cs) ----------------- C1 = C2 = 2(15-5) = 20pF"
- note removed: "Oscillator"
- note removed: "RGB Leds"
- note removed: "Select a ferrite bead"
- moved on the sheet: C36, C37, C38, C4, C41, C43, C44, C5, C56, C59, C6, C63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

Commit message: .
Parts:
- removed R11: 1k, Capacitor_SMD:C_0402_1005Metric, symbol Device:R
- added R83: 1k, Resistor_SMD:R_0402_1005Metric, symbol Device:R
- R10, R15: footprint Capacitor_SMD:C_0402_1005Metric -> Resistor_SMD:R_0402_1005Metric; Distributer Link https://www.ozdisan.com/p/smt-smd-ve-cip-direncler-194/roya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 -> https://www.ozdisan.com/p/smt-smd-ve-cip-direncler-194/pana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; Part Number CQ02WGJ0103TCE -> ERJ2RKF1002X
- R14: footprint Capacitor_SMD:C_0402_1005Metric -> Resistor_SMD:R_0402_1005Metric
- SW1: Distributer Link https://www.e-komponent.com/arama?q=spdt+&category=297 -> https://www.ozdisan.com/p/surgulu-sivicler-495/kls-electron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; Part Number (none) -> L-KLS7-MSK-12C03
- U7: Distributer Link (none) -> https://www.mouser.com.tr/en/ProductDetail/STMicroelectroni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
Connections:
- net GND: now also R83.2
- net at D4.1 (K): now also R83.1
Other:
- note added: "Add buzzer"
- moved on the sheet: C1, C10, C16, C17, C18, C3, C4, C5, C56, C59, C63, C64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

Commit message: .
Parts:
- removed R24: 20, Resistor_SMD:R_0402_1005Metric, symbol Device:R
- removed Y1: 25MHz, Oscillator:Oscillator_SMD_Abracon_ASDMB-4Pin_2.5x2.0mm, symbol Device:Crystal
- added BZ1: Buzzer, footprints:Buzzer_typeshit, symbol Device:Buzzer
- added C32: 2.2uF, Capacitor_SMD:C_0603_1608Metric, symbol Device:C
- added C53: 100nF, Capacitor_SMD:C_0402_1005Metric, symbol Device:C
- added D1, D5, D7: 1N4148, Diode_SMD:D_SOD-523, symbol Diode:1N4148WS
- added Q1: BC847, Package_TO_SOT_SMD:SOT-23, symbol Transistor_BJT:BC847
- added R1: R, symbol Device:R
- added R106: 22, Resistor_SMD:R_0402_1005Metric, symbol Device:R
- added R84: 1k, Resistor_SMD:R_0402_1005Metric, symbol Device:R
- added Y3: 25MHz, Oscillator:Oscillator_SMD_Abracon_ASDMB-4Pin_2.5x2.0mm, symbol Device:Crystal_GND24_Small
- Y2: footprint Crystal:Crystal_SMD_2012-2Pin_2.0x1.2mm_HandSoldering -> Crystal:Crystal_SMD_2012-2Pin_2.0x1.2mm
Connections:
- net +3.3V: now also R106.1
- net Buzzer: now also R84.2
- net GND: now also C32.2, C53.2, Y3.2, Y3.4
- net OSC_IN: now also Y3.3
- net OSC_OUT: now also Y3.1
- net VREF+: now also R106.2
- new net: D5.1 (K), R1.1
- new net: D1.1 (K), D5.2 (A)
- new net: BZ1.1 (+), D7.1 (K), R1.2
- new net: BZ1.2 (-), D7.2 (A), Q1.3 (C)
- new net: Q1.1 (B), R84.1
- new net +5VP: C32.1, C53.1, D1.2 (A)
Other:
- note added: "Buzzer"
- note removed: "Add buzzer"
- moved on the sheet: C1, C16, C3, C4, D4, D6, R14, R83, Y2

Commit message: .
Parts:
- R1: value R -> 22; footprint (none) -> Resistor_SMD:R_0603_1608Metric; Distributer Link (none) -> https://www.ozdisan.com/p/smt-smd-ve-cip-direncler-194/pana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; Part Number (none) -> ERJPA3J220V
Changed lines of the file:
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@@
 			)
 		)
-		(property "Value" "R"
+		(property "Value" "22"
 			(at 209.042 128.27 90)
 			(show_name no)
@@
 			)
 		)
-		(property "Footprint" ""
+		(property "Footprint" "Resistor_SMD:R_0603_1608Metric"
 			(at 209.042 133.096 90)
 			(hide yes)
@@
 			)
 		)
-		(property "Datasheet" ""
+		(property "Datasheet" "https://cdn.ozdisan.com/public/product/assets/Pansonic_Anti-Sulfurated%20Thick%20Film%20Chip%20Resistors_ERJ-S%2CS02%2CS03%2CS06%2CS08%2CS14%2CS12%2CS1D%2CS1T%2CU%2CU0X%2CU01%2CU03%2CU06%2CU08%2CU14%2CU12%2CU1D%2CU1T%2CU6S%2CU6Q_Series_AOA0000C334.pdf?response-content-type=application%2Fpdf&response-content-disposition=inline"
 			(at 209.042 131.318 0)
 			(hide yes)
@@
 			)
 		)
-		(property "Description" "Resistor"
+		(property "Description" "RES.(1608) 0603 22 Ohms 5% 1/3W 200PPM AECQ200"
 			(at 209.042 131.318 0)
 			(hide yes)
+			(show_name no)
+			(do_not_autoplace no)
+			(effects
+				(font
+					(size 1.27 1.27)
+				)
+			)
+		)
+		(property "Distributer Link" "https://www.ozdisan.com/p/smt-smd-ve-cip-direncler-194/panasoniceurope-erjpa3j220v-1189964?catSequenceId=194"
+			(at 209.042 131.318 0)
+			(hide yes)
+			(show_name no)
+			(do_not_autoplace no)
+			(effects
+				(font
+					(size 1.27 1.27)
+				)
+			)
+		)
+		(property "Part Number" "ERJPA3J220V"
+			(at 209.042 131.318 0)
+			(hide yes)

Commit message: .
Connections:
- net OSC_IN: now also C16.1, Y3.1; no longer C4.1, Y3.3
- net OSC_OUT: now also C4.1, Y3.3; no longer C16.1, Y3.1
- net VCAP1: now reaches C5.2, U7.48 (VCAP)
- net VCAP2: now reaches C10.2, U7.73 (VCAP)
- no-connect marks 16 -> 17
Changed lines of the file:
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@@
 	)
 	(no_connect
+		(at 128.524 99.568)
+	)
+	(no_connect
 		(at 128.524 76.708)
 	)
@@
 		)
 	)
+	(label "VCAP2"
+		(at 82.042 163.068 180)
+		(effects
+			(font
+				(size 1.27 1.27)
+			)
+			(justify right bottom)
+		)
+	)
 	(label "BLUE_LED"
 		(at 128.524 140.208 0)
@@
 		)
 	)
+	(label "VCAP1"
+		(at 75.946 160.528 0)
+		(effects
+			(font
+				(size 1.27 1.27)
+			)
+			(justify left bottom)
+		)
+	)
 	(label "BLUE_LED"
 		(at 34.544 117.348 0)
@@
 	)
 	(label "OSC_IN"
-		(at 23.622 65.278 180)
+		(at 35.306 64.77 0)
 		(effects
 			(font
 				(size 1.27 1.27)
 			)
-			(justify right bottom)
+			(justify left bottom)
 		)
 	)
@@
 	)
 	(label "OSC_OUT"
-		(at 35.306 65.786 0)
+		(at 23.622 64.77 180)
 		(effects
 			(font
 				(size 1.27 1.27)
 			)
-			(justify left bottom)
+			(justify right bottom)
 		)
 	)
