File: Ahrar Flight Controller/Power.kicad_sch (KiCad schematic)
At the start: 38 parts, among them J11 Conn_01x06, J9 USB4105-GF-A-120, U1 TPS562200, U2 AP2112K-3.3TRG1, U4 TPD2EUSB30DRTR, U8 TPS2121RUXR

Commit message: Adding previous files
Parts:
- removed D10: PTVS5V0P1UP, Diode_SMD:D_SOD-128, symbol Device:D_Zener
- added D3: ESD321DYAR, Diode_SMD:D_SOD-523, symbol Diode:ESD5Zxx
Connections:
- net GND: now also D3.2 (A)
- net VBUS: now also D3.1 (K)
Other:
- note added: "- Consider single LDO with big footprint to dissipate power and better regulation - RC filter on ADC lines"
- note added: "Current estimation for 3.3V handling: - MCU -> 300mA -> Buck - IMU -> 0.88 mA -> LDO - BARO -> 1.4 mA (peak)-> LDO - GPS & Compass connection -> 50mA -> LDO - SD-card -> 20-100 mA (working) 200-300mA max -> Buck ------------------------ Worst case senario - Buck = 500mA Worst case senario - LDO = 80mA Worst case senario = 680mA - 700mA ++++======================++++ Current estimation for 5V hand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"
- note removed: "- Power Mux - USB-c impedence matching - LDO current and power dissipation values"
- note removed: "- Power mux - USB-c - finalize the LDOs - Input voltage from PDB"
- note removed: "Current limiting"

Commit message: .
Parts:
- removed C14, C15: 22uF, Capacitor_SMD:C_0603_1608Metric, symbol Device:C
- removed C2, C8: 10uF, Capacitor_SMD:C_1206_3216Metric, symbol Device:C
- removed C29, C33, C35: 1uF, Capacitor_SMD:C_0402_1005Metric, symbol Device:C
- removed C30: 10uF, Capacitor_SMD:C_0805_2012Metric, symbol Device:C
- removed C60, C61, C62, C68, C69: 100nF, Capacitor_SMD:C_0402_1005Metric, symbol Device:C
- removed D2: RED_LED, Capacitor_SMD:C_0402_1005Metric, symbol Device:LED
- removed D3: ESD321DYAR, Diode_SMD:D_SOD-523, symbol Diode:ESD5Zxx
- removed FB2, FB3: FerriteBead, Resistor_SMD:R_0805_2012Metric, symbol Device:FerriteBead
- removed J11: Conn_01x06, footprints.5024430670:CONN_502443-06xx_MOL, symbol Connector_Generic:Conn_01x06
- removed J9: USB4105-GF-A-120, USB4105-GF-A-120:GCT_USB4105-GF-A-120, symbol USB4105-GF-A-120:USB4105-GF-A-120
- removed L1: 3.3uH, WE-TPC_4828:WE-TPC_4828, symbol Device:L
- removed R13, R5: 5.1k, Capacitor_SMD:C_0402_1005Metric, symbol Device:R
- removed R41: 33.2k, Capacitor_SMD:C_0402_1005Metric, symbol Device:R
- removed R6: 1k, Capacitor_SMD:C_0402_1005Metric, symbol Device:R
- removed R8: 10kΩ, Resistor_SMD:R_0603_1608Metric, symbol Device:R
- removed U1: TPS562200, Package_TO_SOT_SMD:SOT-23-6, symbol Regulator_Switching:TPS562200
- removed U2: AP2112K-3.3TRG1, AP2112K-3.3TRG1:SOT95P285X140-5N, symbol AP2112K-3.3TRG1:AP2112K-3.3TRG1
- removed U4: TPD2EUSB30DRTR, Package_TO_SOT_SMD:Texas_DRT-3, symbol Power_Protection:TPD2EUSB30A
- added C11: 22uF, Capacitor_SMD:C_0805_2012Metric, symbol Device:C
- added C74, C75: 100nF, Capacitor_SMD:C_0402_1005Metric, symbol Device:C
- added J17: Conn_01x06, Connector_Molex:Molex_CLIK-Mate_502494-0670_1x06-1MP_P2.00mm_Horizontal, symbol Connector_Generic:Conn_01x06
- added R4, R9: 4.7, Resistor_SMD:R_0402_1005Metric, symbol Device:R
Connections:
- net +5V: now also C11.1, J17.1 (Pin_1), J17.2 (Pin_2)
- net Current_sense: now also R4.2
- net GND: now also C11.2, C74.2, C75.2, J17.5 (Pin_5), J17.6 (Pin_6)
- net Voltage_sense: now also R9.2
- new net Current_Connection: C74.1, J17.3 (Pin_3), R4.1
- new net Voltage_Connection: C75.1, J17.4 (Pin_4), R9.1
- no-connect marks 2 -> 0
Other:
- note added: "- Consider single LDO with big footprint to dissipate power and better regulation"
- note added: "RC Filters For ADC Pins"
- note removed: "- Consider single LDO with big footprint to dissipate power and better regulation - RC filter on ADC lines"
- note removed: "USB-c"
- moved on the sheet: C48, C67, R2, R35, R37, R39, R40, R42, R7, U8

Commit message: .
Parts:
- removed C48: 1uF, Capacitor_SMD:C_0402_1005Metric, symbol Device:C
- removed R7: 10kΩ, Resistor_SMD:R_0603_1608Metric, symbol Device:R
- added C22, C30: 2.2uF, Capacitor_SMD:C_0603_1608Metric, symbol Device:C
- added C40, C69: 100nF, Capacitor_SMD:C_0402_1005Metric, symbol Device:C
- added C8: 22uF, Capacitor_SMD:C_0805_2012Metric, symbol Device:C
- added R50: 10kΩ, Resistor_SMD:R_0402_1005Metric, symbol Device:R
- added U2: TLV1117-33, Package_SON:WSON-8-1EP_4x4mm_P0.8mm_EP2.2x3mm, symbol Regulator_Linear:TLV1117-33
- R35, R39, R42: footprint Capacitor_SMD:C_0402_1005Metric -> Resistor_SMD:R_0402_1005Metric
- U8: value TPS2121RUXR -> TPS2121; Distributer Link (none) -> https://www.mouser.com.tr/en/ProductDetail/Texas-Instrument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; Part Number (none) -> TPS2121RUXR
Connections:
- net GND: now also C22.2, C30.2, C40.2, C69.2, C8.2, R50.1, U2.1 (ADJ/GND), U2.8 (NC)
- net VCC: now also C22.1, C69.1, U2.2 (Vin), U2.3 (Vin), U2.4 (Vin)
- net at R35.2, U8.6 (PR1): now also R50.2
- net at U8.11 (SS): now also C30.1
- new net +3.3V: C40.1, C8.1, U2.5 (Vout), U2.6 (Vout), U2.7 (Vout)
Other:
- note added: "LDO"
- moved on the sheet: C11, C67, C74, C75, J17, R2, R35, R37, R39, R4, R42, R9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

Commit message: .
Parts:
- removed J17: Conn_01x06, Connector_Molex:Molex_CLIK-Mate_502494-0670_1x06-1MP_P2.00mm_Horizontal, symbol Connector_Generic:Conn_01x06
- added J10: Conn_01x06_MountingPin, Connector_Molex:Molex_CLIK-Mate_502494-0670_1x06-1MP_P2.00mm_Horizontal, symbol Connector_Generic_MountingPin:Conn_01x06_MountingPin
Connections:
- net +5V: now also J10.1 (Pin_1), J10.2 (Pin_2)
- net Current_Connection: now also J10.3 (Pin_3)
- net GND: now also U2.9 (PAD), J10.5 (Pin_5), J10.6 (Pin_6), J10.MP (MountPin)
- net Voltage_Connection: now also J10.4 (Pin_4)
- net VCC renamed +5VP
Other:
- note removed: "- Consider single LDO with big footprint to dissipate power and better regulation"
- note removed: "Current estimation for 3.3V handling: - MCU -> 300mA -> Buck - IMU -> 0.88 mA -> LDO - BARO -> 1.4 mA (peak)-> LDO - GPS & Compass connection -> 50mA -> LDO - SD-card -> 20-100 mA (working) 200-300mA max -> Buck ------------------------ Worst case senario - Buck = 500mA Worst case senario - LDO = 80mA Worst case senario = 680mA - 700mA ++++======================++++ Current estimation for 5V hand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"
- moved on the sheet: C11, C22, C30, C40, C67, C69, C74, C75, C8, R2, R35, R37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

Commit message: .
Parts:
- removed C67: 100nF, Capacitor_SMD:C_0402_1005Metric, symbol Device:C
