File: Ahrar Flight Controller/Sensors.kicad_sch (KiCad schematic)
At the start: 7 parts, among them U3 MS5611-01BA

Commit message: Adding previous files
Other:
- note added: "BMP388"
- note added: "ICM-42688"
- note added: "ICM-45686"
- note added: "MS5611"
- note removed: "Baro-temperature"
- note removed: "IMU-GYRO"
Changed lines of the file:
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@@
 		(comment 1 "Ahrar Team")
 	)
-	(text "Baro-temperature"
+	(text "MS5611\n"
 		(exclude_from_sim no)
-		(at 174.498 42.418 0)
+		(at 148.336 41.91 0)
+		(effects
+			(font
+				(size 3.81 3.81)
+				(thickness 0.762)
+				(bold yes)
+			)
+			(justify left)
+		)
+	)
+	(text "BMP388"
+		(exclude_from_sim no)
+		(at 159.512 110.49 0)
 		(effects
 			(font
@@
 		)
 	)
-	(text "IMU-GYRO"
+	(text "ICM-42688"
+		(exclude_from_sim no)
+		(at 44.704 42.672 0)
+		(effects
+			(font
+				(size 3.81 3.81)
+				(thickness 0.762)
+				(bold yes)
+			)
+		)
+	)
+	(text "ICM-45686"
 		(exclude_from_sim no)
-		(at 44.45 42.926 0)
+		(at 45.212 110.998 0)
 		(effects
 			(font
@@
 		)
 	)
+	(global_label "BARO_SPI_MOSI"
+		(shape bidirectional)
+		(at 234.442 92.202 0)
+		(fields_autoplaced yes)
+		(effects
+			(font
+				(size 1.27 1.27)
+				(thickness 0.254)
+				(bold yes)
+			)
+			(justify left)
+		)
+		(property "Intersheetrefs" "${INTERSHEET_REFS}"
+			(at 253.5893 92.202 0)
+			(hide yes)
+			(show_name no)
+			(do_not_autoplace no)
+			(effects
+				(font
+					(size 1.27 1.27)
+				)
+				(justify left)
+			)
+		)
+	)
+	(global_label "BARO_SPI_MISO"
+		(shape bidirectional)
+		(at 234.95 88.9 0)
+		(fields_autoplaced yes)
+		(effects
+			(font
+				(size 1.27 1.27)
+				(thickness 0.254)
+				(bold yes)
+			)
+			(justify left)
+		)
+		(property "Intersheetrefs" "${INTERSHEET_REFS}"
+			(at 254.0973 88.9 0)
+			(hide yes)
+			(show_name no)
+			(do_not_autoplace no)
+			(effects
+				(font
+					(size 1.27 1.27)
+				)
+				(justify left)
+			)
+		)
+	)
+	(global_label "BARO_SPI_CLK"
+		(shape input)
+		(at 216.408 92.456 0)
+		(fields_autoplaced yes)
+		(effects
+			(font
+				(size 1.27 1.27)
+				(thickness 0.254)
+				(bold yes)
+			)
+			(justify left)
+		)
+		(property "Intersheetrefs" "${INTERSHEET_REFS}"
+			(at 233.4159 92.456 0)
+			(hide yes)
+			(show_name no)
+			(do_not_autoplace no)
+			(effects
+				(font
+					(size 1.27 1.27)
+				)
+				(justify left)
+			)
+		)
+	)
+	(global_label "BARO_SPI_SS"
+		(shape input)
+		(at 238.252 96.012 0)
+		(fields_autoplaced yes)
+		(effects
+			(font
+				(size 1.27 1.27)
+				(thickness 0.254)
+				(bold yes)
+			)
+			(justify left)
+		)
+		(property "Intersheetrefs" "${INTERSHEET_REFS}"
+			(at 254.1108 96.012 0)
+			(hide yes)
+			(show_name no)
+			(do_not_autoplace no)
+			(effects
+				(font
+					(size 1.27 1.27)
+				)
+				(justify left)
+			)
+		)
+	)
 	(hierarchical_label "IMU_INT"
 		(shape input)
@@
 			)
 			(stroke
+				(width 0)
+				(type dash)
+			)
+			(fill
+				(type none)
+			)
+		)
+	)
+	(rule_area
+		(exclude_from_sim no)
+		(in_bom yes)
+		(on_board yes)
+		(dnp no)
+		(polyline
+			(pts
+				(xy 27.178 105.664) (xy 27.178 174.244) (xy 146.558 174.244) (xy 146.558 106.934) (xy 146.558 105.41)
+			)
+			(stroke
+				(width 0)
+				(type dash)
+			)
+			(fill
+				(type none)
+			)
+		)
+	)
+	(rule_area
+		(exclude_from_sim no)
+		(in_bom yes)
+		(on_board yes)
+		(dnp no)
+		(polyline
+			(pts
+				(xy 146.558 105.664) (xy 146.558 174.244) (xy 265.938 174.244) (xy 265.938 106.934) (xy 265.938 105.41)
+			)
+			(stroke

Commit message: .
Parts:
- removed C31: 1uF, Capacitor_SMD:C_0402_1005Metric, symbol Device:C
- added C19, C20, C21: 2.2uF, Capacitor_SMD:C_0603_1608Metric, symbol Device:C
- added C70, C71, C72, C73: 100nF, Capacitor_SMD:C_0402_1005Metric, symbol Device:C
- added MT2: ICM-45686, ICM_42688_P:LGA14_2P5X3X0P91_TDK-L, symbol ICM-42670-P:ICM-42670-P
- added R12, R17, R25, R26, R27, R3, R38, R43, R44, R47, R48, R49: 20, Resistor_SMD:R_0402_1005Metric, symbol Device:R
- added R36, R45, R46, R50: 10kΩ, Capacitor_SMD:C_0402_1005Metric, symbol Device:R
- added R56, R77, R78: 220, Resistor_SMD:R_0402_1005Metric, symbol Device:R
- added U5: BMP581, BMP581:BMP581, symbol IR2103STRPBF:BMP380
Connections:
- net GND: now also MT1.10 (RESV__2), MT1.11 (RESV__3), MT1.2 (RESV), MT1.3 (RESV__1), MT1.7 (RES), C19.2, C20.2, C21.2, C70.2, C71.2, C72.2, C73.2, MT2.10 (RESV__2), MT2.11 (RESV__3), MT2.2 (RESV), MT2.3 (RESV__1), MT2.6 (GND), MT2.7 (RESV), U5.3 (GND), U5.8 (GND), U5.9 (GND)
- net +3.3VA renamed +3.3V
- net +3.3V: now also C19.1, C20.1, C21.1, C70.1, C71.1, C72.1, C73.1, MT2.5 (VDDIO), MT2.8 (VDD), R36.1, R45.1, R46.1, R50.1, U5.1 (VDDIO), U5.10 (VDD)
- net BARO_SPI_MISO: no longer names the net of U3.6 (SDO)
- net BARO_SPI_MISO: now also R47.2
- net BARO_SPI_MOSI: no longer names the net of U3.7 (SDI/SDA)
- net BARO_SPI_MOSI: now also R48.2
- net BARO_SPI_SCLK: no longer names the net of U3.8 (SCLK)
- net BARO_SPI_SCLK: now also R49.2
- net BARO_SPI_SS renamed MS_SPI_SS
- net MS_SPI_SS: now also R46.2
- net IMU_INT: no longer names the net of MT1.4 (INT1/INT)
- net IMU_INT: now also R56.1
- net IMU_SPI_MISO: no longer names the net of MT1.1 (AP_SDO/AP_AD0)
- net IMU_SPI_MISO: now also R25.2
- net IMU_SPI_MOSI: no longer names the net of MT1.14 (AP_SDA/AP_SDIO/AP_SDI)
- net IMU_SPI_MOSI: now also R17.2
- net IMU_SPI_SCLK: no longer names the net of MT1.13 (AP_SCL/AP_SCLK)
- net IMU_SPI_SCLK: now also R12.2
- net IMU_SPI_SS renamed ICM88_SS
- net ICM88_SS: now also R50.2
- new net: R43.2, U5.4 (SDI)
- new net: MT2.13 (AP_SCL/AP_SCLK), R26.2
- new net: MT2.1 (AP_SDO/AP_AD0), R27.2
- new net: MT2.14 (AP_SDA/AP_SDIO/AP_SDI), R3.2
- new net: MT2.4 (INT1/INT), R77.1
- new net: R38.2, U5.2 (SCK)
- new net: R44.2, U5.5 (SDO)
- new net: R78.1, U5.7 (INT)
- new net BMP_INT: R78.2
- new net BMP_MISO: R44.1
- new net BMP_MOSI: R43.1
- new net BMP_SCK: R38.1
- new net BMP_SS: R45.2, U5.6 (CSB)
- new net ICM86_INT: R77.2
- new net ICM86_MISO: R27.1
- new net ICM86_MOSI: R3.1
- new net ICM86_SCLK: R26.1
- new net ICM86_SS: MT2.12 (AP_CS), R36.2
- new net ICM88_INT: R56.2
- new net ICM88_MISO: R25.1
- new net ICM88_MOSI: R17.1
- new net ICM88_SCK: R12.1
- new net MS_SPI_CLK: R49.1
- new net MS_SPI_MISO: R47.1
- new net MS_SPI_MOSI: R48.1
- no-connect marks 6 -> 2
Other:
- note added: "BMP581"
- note added: "Max current consumption: 0.26mA"
- note added: "Max current consumption: 0.42mA"
- note added: "Max current consumption: 0.88mA"
- note added: "Max current consumption: 1.4mA"
- note removed: "BMP388"
- note removed: "Use SPI"
- moved on the sheet: C13, C58, C65, C66, MT1, U3

Commit message: .
Parts:
- removed R50: 10kΩ, Capacitor_SMD:C_0402_1005Metric, symbol Device:R
- added R41: 10kΩ, Resistor_SMD:R_0402_1005Metric, symbol Device:R
- added R79, R80, R81, R82: 20, Resistor_SMD:R_0402_1005Metric, symbol Device:R
- R36, R45, R46: footprint Capacitor_SMD:C_0402_1005Metric -> Resistor_SMD:R_0402_1005Metric; Distributer Link https://www.ozdisan.com/p/smt-smd-ve-cip-direncler-194/roya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 -> https://www.ozdisan.com/p/smt-smd-ve-cip-direncler-194/pana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; Part Number CQ02WGJ0103TCE -> ERJ2RKF1002X
Connections:
- net +3.3V: now also R41.1
- net BMP_SS: now also R79.1; no longer U5.6 (CSB)
- net ICM86_SS: now also R82.1; no longer MT2.12 (AP_CS)
- net ICM88_SS: now also R41.2, R81.1; no longer MT1.12 (AP_CS)
- net MS_SPI_SS: now also R80.1; no longer U3.4 (CSB), U3.5 (CSB)
- new net: MT2.12 (AP_CS), R82.2
- new net: R79.2, U5.6 (CSB)
- new net: MT1.12 (AP_CS), R81.2
- new net: R80.2, U3.4 (CSB), U3.5 (CSB)

Commit message: .
Parts:
- removed R12, R17, R25, R26, R27, R3, R38, R43, R44, R47, R48, R49, R79, R80, R81: 20, Resistor_SMD:R_0402_1005Metric, symbol Device:R
- added R100, R86, R87, R88, R89, R90, R91, R92, R93, R94, R95, R96, R97, R98, R99: 22, Resistor_SMD:R_0402_1005Metric, symbol Device:R
- R82: value 20 -> 22; Distributer Link https://www.ozdisan.com/p/smt-smd-ve-cip-direncler-194/pana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 -> https://www.ozdisan.com/p/smt-smd-ve-cip-direncler-194/roya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; Part Number ERJ2GEJ200X -> CQ02WGF220JTCE
Connections:
- net BMP_MISO: now also R91.1
- net BMP_MOSI: now also R90.1
- net BMP_SCK: now also R89.1
- net BMP_SS: now also R92.1; no longer R45.2
- net ICM86_MISO: now also R88.1
- net ICM86_MOSI: now also R87.1
- net ICM86_SCLK: now also R86.1
- net ICM86_SS: no longer R36.2
- net ICM88_MISO: now also R100.1
- net ICM88_MOSI: now also R99.1
- net ICM88_SCK: now also R98.1
- net ICM88_SS: now also R97.1; no longer R41.2
- net MS_SPI_CLK: now also R95.1
- net MS_SPI_MISO: now also R93.1
- net MS_SPI_MOSI: now also R94.1
- net MS_SPI_SS: now also R96.1; no longer R46.2
- net at U5.4 (SDI): now also R90.2
- net at MT2.13 (AP_SCL/AP_SCLK): now also R86.2
- net at MT2.1 (AP_SDO/AP_AD0): now also R88.2
- net at MT2.12 (AP_CS), R82.2: now also R36.2
- net at MT2.14 (AP_SDA/AP_SDIO/AP_SDI): now also R87.2
- net at U5.2 (SCK): now also R89.2
- net at U3.7 (SDI/SDA): now also R94.2
- net at MT1.1 (AP_SDO/AP_AD0): now also R100.2
- net at U5.5 (SDO): now also R91.2
- net at MT1.14 (AP_SDA/AP_SDIO/AP_SDI): now also R99.2
- net at U5.6 (CSB): now also R45.2, R92.2
- net at MT1.12 (AP_CS): now also R41.2, R97.2
- net at MT1.13 (AP_SCL/AP_SCLK): now also R98.2
- net at U3.6 (SDO): now also R93.2
- net at U3.4 (CSB), U3.5 (CSB): now also R46.2, R96.2
- net at U3.8 (SCLK): now also R95.2
Other:
- moved on the sheet: C19, C70, C71, R36, R41, R45, R46, R78, R82, U5

Commit message: .
Parts:
- removed C13: 2.2uF, Capacitor_SMD:C_0402_1005Metric, symbol Device:C
- added C33: 2.2uF, Capacitor_SMD:C_0603_1608Metric, symbol Device:C
Connections:
- net +3.3V: now also C33.1
- net GND: now also C33.2
Other:
- moved on the sheet: C72
